File: Subsystem Circuits/Microcontroller.kicad_sch (KiCad schematic)
At the start: 0 parts

Commit message: stuff
Parts:
- added U1: ~, symbol EEE4113F:ESP32-Cam
- added U2: ~, symbol EEE4113F:315MHz-RF-Receiver
- added U3: ~, symbol EEE4113F:315MHz-RF-Transmitter
Connections:
- new net 3V3: U1.16 (3V3)
Changed lines of the file:
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@@
 	(generator_version "8.0")
 	(paper "A4")
+	(hierarchical_label "3V3"
+		(shape input)
+		(at 215.9 121.92 0)
+		(fields_autoplaced yes)
+		(effects
+			(font
+				(size 1.27 1.27)
+			)
+			(justify left)
+		)
+	)
+	(symbol
+		(lib_id "EEE4113F:ESP32-Cam")
+		(at 204.47 130.81 0)
+		(unit 1)
+		(exclude_from_sim no)
+		(in_bom yes)
+		(on_board yes)
+		(dnp no)
+		(fields_autoplaced yes)
+		(property "Reference" "U1"
+			(at 204.47 116.84 0)
+			(effects
+				(font
+					(size 1.27 1.27)
+				)
+			)
+		)
+		(property "Value" "~"
+			(at 204.47 118.11 0)
+			(effects
+				(font
+					(size 1.27 1.27)
+				)
+			)
+		)
+		(property "Footprint" ""
+			(at 201.93 128.27 0)
+			(effects
+				(font
+					(size 1.27 1.27)
+				)
+				(hide yes)
+			)
+		)
+		(property "Datasheet" ""
+			(at 201.93 128.27 0)
+			(effects
+				(font
+					(size 1.27 1.27)
+				)
+				(hide yes)
+			)
+		)
+		(property "Description" ""
+			(at 201.93 128.27 0)
+			(effects
+				(font
+					(size 1.27 1.27)
+				)
+				(hide yes)
+			)
+		)
+		(pin "7"
+		)
+		(pin "13"
+		)
+		(pin "15"
+		)
+		(pin "2"
+		)
+		(pin "8"
+		)
+		(pin "16"
+		)
+		(pin "12"
+		)
+		(pin "9"
+		)
+		(pin "4"
+		)
+		(pin "1"
+		)
+		(pin "11"
+		)
+		(pin "14"
+		)
+		(pin "10"
+		)
+		(pin "3"
+		)
+		(pin "5"
+		)
+		(pin "6"
+		)
+		(instances
+			(project "Subsystem Circuits"
+				(path "/afe21291-0891-4f3f-8ac9-75a73c3559e3/ac52e79b-a2c2-4369-8875-88d7b7108f3b"
+					(reference "U1")
+					(unit 1)
+				)
+			)
+		)
+	)
+	(symbol
+		(lib_id "EEE4113F:315MHz-RF-Transmitter")
+		(at 138.43 137.16 0)
+		(mirror y)
+		(unit 1)
+		(exclude_from_sim no)
+		(in_bom yes)
+		(on_board yes)
+		(dnp no)
+		(property "Reference" "U3"
+			(at 138.176 129.54 0)
+			(effects
+				(font
+					(size 1.27 1.27)
+				)
+			)
+		)
+		(property "Value" "~"
+			(at 138.176 132.08 0)
+			(effects
+				(font
+					(size 1.27 1.27)
+				)
+			)
+		)
+		(property "Footprint" ""
+			(at 140.97 137.16 0)
+			(effects
+				(font
+					(size 1.27 1.27)
+				)
+				(hide yes)
+			)
+		)
+		(property "Datasheet" ""
+			(at 140.97 137.16 0)
+			(effects
+				(font
+					(size 1.27 1.27)
+				)
+				(hide yes)
+			)
+		)
+		(property "Description" ""
+			(at 140.97 137.16 0)
+			(effects
+				(font
+					(size 1.27 1.27)
+				)
+				(hide yes)
+			)
+		)
+		(pin "2"
+		)
+		(pin "3"
+		)
+		(pin "1"
+		)
+		(instances
+			(project "Subsystem Circuits"
+				(path "/afe21291-0891-4f3f-8ac9-75a73c3559e3/ac52e79b-a2c2-4369-8875-88d7b7108f3b"
+					(reference "U3")
+					(unit 1)
+				)
+			)
+		)
+	)
+	(symbol
+		(lib_id "EEE4113F:315MHz-RF-Receiver")
+		(at 161.29 137.16 0)
+		(unit 1)
+		(exclude_from_sim no)
+		(in_bom yes)
+		(on_board yes)
+		(dnp no)
+		(property "Reference" "U2"
+			(at 161.544 128.27 0)
+			(effects
+				(font
+					(size 1.27 1.27)
+				)
+			)
+		)
+		(property "Value" "~"
+			(at 161.544 130.81 0)
+			(effects
+				(font
+					(size 1.27 1.27)
+				)
+			)
+		)
+		(property "Footprint" ""
+			(at 162.56 137.16 0)
+			(effects
+				(font
+					(size 1.27 1.27)
+				)
+				(hide yes)
+			)
+		)
+		(property "Datasheet" ""
+			(at 162.56 137.16 0)
+			(effects
+				(font
+					(size 1.27 1.27)
+				)
+				(hide yes)
+			)
+		)
+		(property "Description" ""
+			(at 162.56 137.16 0)
+			(effects
+				(font
+					(size 1.27 1.27)
+				)
+				(hide yes)
+			)
+		)
+		(pin "3"
+		)
+		(pin "1"
+		)
+		(pin "4"
+		)
+		(pin "2"
+		)
+		(instances
+			(project "Subsystem Circuits"
+				(path "/afe21291-0891-4f3f-8ac9-75a73c3559e3/ac52e79b-a2c2-4369-8875-88d7b7108f3b"
+					(reference "U2")
+					(unit 1)
+				)
+			)
+		)
+	)
 )
